Commit message: Changed camera position and added lidar

File: car_description/urdf/car.xacro (robot description, xacro)
@@ -14,4 +14,6 @@
     <xacro:property name="cameraSize" value="0.05"/>
     <xacro:property name="cameraMass" value="0.1"/>
+    <xacro:property name="laserSize" value="0.05"/>
+    <xacro:property name="laserMass" value="0.1"/>
     <xacro:include filename="$(find car_description)/urdf/car.gazebo" />
     <xacro:include filename="$(find car_description)/urdf/materials.xacro" />
@@ -69,5 +71,5 @@
     <wheel lr="right" tY="-1"/>
     <joint name="camera_joint" type="fixed">
-        <origin xyz="${-cameraSize+chassisLength/2} 0 ${cameraSize+wheelRadius+cameraSize/2}" rpy="0 0 0"/>
+        <origin xyz="${cameraSize+chassisLength/2} 0 ${wheelRadius}" rpy="0 0 0"/>
         <parent link="chassis"/>
         <child link="camera"/>
@@ -93,3 +95,28 @@
         </inertial>
     </link>
+    <joint name="rplidar_joint" type="fixed">
+        <origin xyz="${-laserSize+chassisLength/2} 0 ${wheelRadius+laserSize+laserSize/2}" rpy="0 0 0"/>
+        <parent link="chassis"/>
+        <child link="laser"/>
+    </joint>
+    <link name="laser">
+        <collision>
+            <origin xyz="0 0 0" rpy="0 0 0"/>
+            <geometry>
+                <box size="${laserSize} ${laserSize} ${laserSize}"/>
+            </geometry>
+        </collision>
+        <visual>
+            <origin xyz="0 0 0" rpy="0 0 0"/>
+            <geometry>
+                <box size="${laserSize} ${laserSize} ${laserSize}"/>
+            </geometry>
+            <material name="blue"/>
+        </visual>
+        <inertial>
+            <mass value="${laserSize}"/>
+            <origin xyz="0 0 0" rpy="0 0 0"/>
+            <box_inertia m="${laserSize}" x="${laserSize}" y="${laserSize}" z="${laserSize}"/>
+        </inertial>
+    </link>
 </robot>

Commit message: Fixed typo

File: car_description/urdf/car.xacro (robot description, xacro)
@@ -115,7 +115,7 @@
         </visual>
         <inertial>
-            <mass value="${laserSize}"/>
+            <mass value="${laserMass}"/>
             <origin xyz="0 0 0" rpy="0 0 0"/>
-            <box_inertia m="${laserSize}" x="${laserSize}" y="${laserSize}" z="${laserSize}"/>
+            <box_inertia m="${laserMass}" x="${laserSize}" y="${laserSize}" z="${laserSize}"/>
         </inertial>
     </link>

Commit message: Corrected transforms and frame names
- Corrected frames names for chassis and laser
- Added transform from chassis to laser

File: car_description/urdf/car.xacro (robot description, xacro)
@@ -22,7 +22,7 @@
     <joint name="base_joint" type="fixed">
       <parent link="footprint"/>
-      <child link="chassis"/>
+      <child link="base_link"/>
     </joint>
-    <link name='chassis'>
+    <link name='base_link'>
         <collision>
             <origin xyz="0 0 ${wheelRadius}" rpy="0 0 0"/>
@@ -45,5 +45,5 @@
     </link>
     <joint name="fixed" type="fixed">
-        <parent link="chassis"/>
+        <parent link="base_link"/>
         <child link="caster_wheel"/>
     </joint>
@@ -72,5 +72,5 @@
     <joint name="camera_joint" type="fixed">
         <origin xyz="${cameraSize+chassisLength/2} 0 ${wheelRadius}" rpy="0 0 0"/>
-        <parent link="chassis"/>
+        <parent link="base_link"/>
         <child link="camera"/>
     </joint>
@@ -97,5 +97,5 @@
     <joint name="rplidar_joint" type="fixed">
         <origin xyz="${-laserSize+chassisLength/2} 0 ${wheelRadius+laserSize+laserSize/2}" rpy="0 0 0"/>
-        <parent link="chassis"/>
+        <parent link="base_link"/>
         <child link="laser"/>
     </joint>

File: car_description/urdf/macros.xacro (robot description, xacro)
@@ -46,5 +46,5 @@
         </gazebo>
         <joint name="${lr}_wheel_hinge" type="continuous">
-            <parent link="chassis"/>
+            <parent link="base_link"/>
             <child link="${lr}_wheel"/>
             <origin xyz="${+wheelPos-chassisLength/4} ${tY*wheelWidth/2+tY*chassisWidth/2} ${wheelRadius}" rpy="0 0 0"/>

Commit message: Fixed laser position to void detecting the wheels

File: car_description/urdf/car.xacro (robot description, xacro)
@@ -96,5 +96,5 @@
     </link>
     <joint name="rplidar_joint" type="fixed">
-        <origin xyz="${-laserSize+chassisLength/2} 0 ${wheelRadius+laserSize+laserSize/2}" rpy="0 0 0"/>
+        <origin xyz="${-laserSize/2+chassisLength/2} 0 ${wheelRadius + chassisHeight/2 + 1.5*laserSize}" rpy="0 0 0"/>
         <parent link="base_link"/>
         <child link="laser"/>

Commit message: Added IMU to the car's model

File: car_description/urdf/car.xacro (robot description, xacro)
@@ -16,4 +16,6 @@
     <xacro:property name="laserSize" value="0.05"/>
     <xacro:property name="laserMass" value="0.1"/>
+    <xacro:property name="imuSize" value="0.02"/>
+    <xacro:property name="imuMass" value="0.01"/>
     <xacro:include filename="$(find car_description)/urdf/car.gazebo" />
     <xacro:include filename="$(find car_description)/urdf/materials.xacro" />
@@ -71,5 +73,5 @@
     <wheel lr="right" tY="-1"/>
     <joint name="camera_joint" type="fixed">
-        <origin xyz="${cameraSize+chassisLength/2} 0 ${wheelRadius}" rpy="0 0 0"/>
+        <origin xyz="${cameraSize/2+chassisLength/2} 0 ${wheelRadius}" rpy="0 0 0"/>
         <parent link="base_link"/>
         <child link="camera"/>
@@ -93,4 +95,29 @@
             <origin xyz="0 0 0" rpy="0 0 0"/>
             <box_inertia m="${cameraMass}" x="${cameraSize}" y="${cameraSize}" z="${cameraSize}"/>
+        </inertial>
+    </link>
+    <joint name="imu_joint" type="fixed">
+        <origin xyz="0 0 ${wheelRadius + chassisHeight/2 + 1.5*imuSize}" rpy="0 0 0"/>
+        <parent link="base_link"/>
+        <child link="base_imu_link"/>
+    </joint>
+    <link name="base_imu_link">
+        <collision>
+            <origin xyz="0 0 0" rpy="0 0 0"/>
+            <geometry>
+                <box size="${imuSize} ${imuSize} ${imuSize}"/>
+            </geometry>
+        </collision>
+        <visual>
+            <origin xyz="0 0 0" rpy="0 0 0"/>
+            <geometry>
+                <box size="${imuSize} ${imuSize} ${imuSize}"/>
+            </geometry>
+            <material name="green"/>
+        </visual>
+        <inertial>
+            <mass value="${imuMass}"/>
+            <origin xyz="0 0 0" rpy="0 0 0"/>
+            <box_inertia m="${imuMass}" x="${imuSize}" y="${imuSize}" z="${imuSize}"/>
         </inertial>
     </link>

Commit message: Changes to footprint and odom->footprint transform
- Renamed footprint to base_footprint
- Prevent gazebo to publish odom to base_footprint transform (we want
robot_localization to publish this).

File: car_description/urdf/car.xacro (robot description, xacro)
@@ -21,7 +21,7 @@
     <xacro:include filename="$(find car_description)/urdf/materials.xacro" />
     <xacro:include filename="$(find car_description)/urdf/macros.xacro" />
-    <link name="footprint" />
+    <link name="base_footprint" />
     <joint name="base_joint" type="fixed">
-      <parent link="footprint"/>
+      <parent link="base_footprint"/>
       <child link="base_link"/>
     </joint>

File: car_description/urdf/macros.xacro (robot description, xacro)
@@ -56,5 +56,5 @@
             <type>transmission_interface/SimpleTransmission</type>
             <joint name="${lr}_wheel_hinge">
-                <hardwareInterface>EffortJointInterface</hardwareInterface>
+                <hardwareInterface>hardware_interface/EffortJointInterface</hardwareInterface>
             </joint>
             <actuator name="${lr}Motor">
